File: low_cost_multispectral_sensor/low_cost_multispectral_sensor.sch (KiCad schematic (older format))
At the start: 32 parts, among them J1 USB_B_Micro, J2 GPIO Conn, J4 Programming Header, U1 MCP2221, U2 MIC5219-3.3YMM, U3 TPD2EUSB30, U5 AS726x, U7 AT25SF041

Commit message: fixed resets
Parts:
- added J5: RST Header, symbol Connector_Generic:Conn_01x02
- added R11: 10K, symbol crystals:R
Connections:
- net 3.3V: now also R11.1
- net GND: now also J5.2 (Pin_2)
- net RST: no longer U5.2 (Reset)
- new net AS_RST: J5.1 (Pin_1), R11.2, U5.2 (Reset)
Other:
- note added: "AS726x reset needs to be held\nin reset during programming"
- moved on the sheet: J4
Changed lines of the file:
@@
 Connection ~ 6320 3130
-Wire Wire Line
-	6130 2980 6450 2980
-Text Label 6130 2980 2    50   ~ 0
-RST
 Wire Wire Line
 	6450 2580 6130 2580
@@
 L Connector_Generic:Conn_01x06 J4
 U 1 1 5DBB8346
-P 10560 1040
-F 0 "J4" H 10510 1340 50  0000 L CNN
-F 1 "Programming Header" V 10660 680 50  0000 L CNN
-F 2 "" H 10560 1040 50  0001 C CNN
-F 3 "~" H 10560 1040 50  0001 C CNN
-	1    10560 1040
-	1    0    0    -1
-$EndComp
-Wire Wire Line
-	10360 840  10160 840
-Wire Wire Line
-	10360 940  10160 940
-Wire Wire Line
-	10360 1040 10160 1040
-Wire Wire Line
-	10360 1140 10160 1140
-Wire Wire Line
-	10360 1240 10160 1240
-Wire Wire Line
-	10360 1340 10160 1340
-Text Label 10160 840  2    50   ~ 0
-3.3V
-Text Label 10160 940  2    50   ~ 0
+P 10870 1020
+F 0 "J4" H 10820 1320 50  0000 L CNN
+F 1 "Programming Header" V 10970 660 50  0000 L CNN
+F 2 "" H 10870 1020 50  0001 C CNN
+F 3 "~" H 10870 1020 50  0001 C CNN
+	1    10870 1020
+	1    0    0    -1
+$EndComp
+Wire Wire Line
+	10670 820  10470 820
+Wire Wire Line
+	10670 920  10470 920
+Wire Wire Line
+	10670 1020 10470 1020
+Wire Wire Line
+	10670 1120 10470 1120
+Wire Wire Line
+	10670 1220 10470 1220
+Wire Wire Line
+	10670 1320 10470 1320
+Text Label 10470 820  2    50   ~ 0
+3.3V
+Text Label 10470 920  2    50   ~ 0
 CS
-Text Label 10160 1040 2    50   ~ 0
+Text Label 10470 1020 2    50   ~ 0
 MISO
-Text Label 10160 1140 2    50   ~ 0
+Text Label 10470 1120 2    50   ~ 0
 MOSI
-Text Label 10160 1240 2    50   ~ 0
+Text Label 10470 1220 2    50   ~ 0
 SCK
 $Comp
 L power:GND #PWR?
 U 1 1 5DBD40C6
-P 10160 1410
-F 0 "#PWR?" H 10160 1160 50  0001 C CNN
-F 1 "GND" H 10165 1237 50  0000 C CNN
-F 2 "" H 10160 1410 50  0001 C CNN
-F 3 "" H 10160 1410 50  0001 C CNN
-	1    10160 1410
-	1    0    0    -1
-$EndComp
-Wire Wire Line
-	10160 1410 10160 1340
+P 10470 1390
+F 0 "#PWR?" H 10470 1140 50  0001 C CNN
+F 1 "GND" H 10475 1217 50  0000 C CNN
+F 2 "" H 10470 1390 50  0001 C CNN
+F 3 "" H 10470 1390 50  0001 C CNN
+	1    10470 1390
+	1    0    0    -1
+$EndComp
+Wire Wire Line
+	10470 1390 10470 1320
 Text Label 8520 2720 0    50   ~ 0
 CS
@@
 Text Label 8700 3020 0    50   ~ 0
 SCK
+Text Label 6130 2980 2    50   ~ 0
+AS_RST
+$Comp
+L crystals:R R11
+U 1 1 5DBE7102
+P 5730 2630
+F 0 "R11" H 5770 2640 50  0000 L CNN
+F 1 "10K" V 5730 2570 50  0000 L CNN
+F 2 "" V 5660 2630 50  0001 C CNN
+F 3 "" H 5730 2630 50  0001 C CNN
+	1    5730 2630
+	1    0    0    -1
+$EndComp
+Wire Wire Line
+	5730 2480 5730 2260
+Text Label 5730 2260 0    50   ~ 0
+3.3V
+Wire Wire Line
+	5730 2780 5730 2980
+Wire Wire Line
+	5730 2980 6450 2980
+$Comp
+L Connector_Generic:Conn_01x02 J5
+U 1 1 5DC05F15
+P 10870 1760
+F 0 "J5" H 10830 1850 50  0000 L CNN
+F 1 "RST Header" V 10970 1600 50  0000 L CNN
+F 2 "" H 10870 1760 50  0001 C CNN
+F 3 "~" H 10870 1760 50  0001 C CNN
+	1    10870 1760
+	1    0    0    -1
+$EndComp
+$Comp
+L power:GND #PWR?
+U 1 1 5DC1017A
+P 10470 1920
+F 0 "#PWR?" H 10470 1670 50  0001 C CNN
+F 1 "GND" H 10475 1747 50  0000 C CNN
+F 2 "" H 10470 1920 50  0001 C CNN
+F 3 "" H 10470 1920 50  0001 C CNN
+	1    10470 1920
+	1    0    0    -1
+$EndComp
+Wire Wire Line
+	10470 1920 10470 1860
+Wire Wire Line
+	10470 1860 10670 1860
+Wire Wire Line
+	10670 1760 10470 1760
+Text Label 10470 1760 2    50   ~ 0
+AS_RST
+Text Notes 8980 1810 0    50   ~ 0
+AS726x reset needs to be held\nin reset during programming
 $EndSCHEMATC

Commit message: Updated schematic
Parts:
- removed D5, D6: D, symbol crystals:D
- removed J4: Programming Header, symbol Connector_Generic:Conn_01x06
- removed J5: RST Header, symbol Connector_Generic:Conn_01x02
- removed R5, R6: R, symbol crystals:R
- added C10: 1uF, Capacitors_SMD:C_0402, symbol crystals:C
- added C6: 2.2uF, Capacitors_SMD:C_0402, symbol crystals:C
- added C7: 100nF, Capacitors_SMD:C_0402, symbol crystals:C
- added C8: 10uF, Capacitors_SMD:C_0402, symbol crystals:C
- added D5, D6: LED, Diodes_SMD:D_1206, symbol crystals:LED
- added D7: D_TVS, Diodes_SMD:D_SMA, symbol Device:D_TVS
- added D8: ESDA6V1-5SC6, Package_TO_SOT_SMD:SOT-23-6, symbol Power_Protection:ESDA6V1-5SC6
- added J3: Flash Programming Header, Pin_Headers:Pin_Header_Straight_2x06_Pitch2.00mm, symbol Connector_Generic:Conn_02x05_Counter_Clockwise
- C1: value C -> 1uF; footprint (none) -> Capacitors_SMD:C_0402
- C2: value C -> 470pF; footprint (none) -> Capacitors_SMD:C_0402
- C3: value C -> 4.7uF; footprint (none) -> Capacitors_SMD:C_0402
- C4: value C -> 0.33uF; footprint (none) -> Capacitors_SMD:C_0402
- C5: footprint (none) -> Capacitors_SMD:C_0402
- D1, D2: footprint (none) -> Diodes_SMD:D_1206
- D3: footprint (none) -> Diodes_SMD:D_SMA
- D4: footprint (none) -> Diodes_SMD:D_SMB
- J1: footprint (none) -> Connectors_USB:USB_Micro-B_Molex-105017-0001
- J2: footprint (none) -> Pin_Headers:Pin_Header_Straight_1x04_Pitch2.54mm
- JP1, JP2, JP3, R1, R11, R2, R3, R4: footprint (none) -> Resistors_SMD:R_0402
- R10, R7, R8, R9: value R -> 10K; footprint (none) -> Resistors_SMD:R_0402
- U1: footprint (none) -> SMD_Packages:SOIC-14_N
- U7: footprint (none) -> SMD_Packages:SOIC-8-N
Connections:
- net 3.3V: now also C10.1, C6.1, C7.1, C8.1, D5.2 (A), D6.2 (A), D7.1 (A1), J3.10 (Pin_10)
- net AS_RST: now also D8.1 (IO1), J3.4 (Pin_4)
- net CS: now also D8.6 (IO5), J3.6 (Pin_6)
- net GND: now also C10.2, C6.2, C7.2, C8.2, D7.2 (A2), D8.2 (GND), J3.1 (Pin_1), J3.2 (Pin_2), J3.3 (Pin_3), J3.5 (Pin_5)
- net MISO: now also D8.3 (IO2), J3.9 (Pin_9)
- net MOSI: now also D8.4 (IO3), J3.8 (Pin_8)
- net SCK: now also D8.5 (IO4), J3.7 (Pin_7)
- net at U5.15 (LED_DRV): now also D6.1 (K)
- net at U5.18 (LED_IND): now also D5.1 (K)
Other:
- moved on the sheet: C1, D3, D4, JP3, R10, R11, R7, R8, R9, U5, U7
