File: low_cost_multispectral_sensor/low_cost_multispectral_sensor.sch (KiCad schematic (older format))
At the start: 41 parts, among them J1 USB_B_Micro, J2 GPIO Conn, J3 Flash Programming Header, U1 MCP2221, U2 MIC5219-3.3YMM, U3 TPD2EUSB30, U5 AS726x, U7 AT25SF041

Commit message: update
Parts:
- H1, H2, H3, H4: footprint (none) -> Mounting_Holes:MountingHole_2.2mm_M2_Pad; symbol Mechanical:MountingHole -> Mechanical:MountingHole_Pad
Connections:
- net GND: now also H1.1, H2.1, H3.1, H4.1
Changed lines of the file:
@@
 	9520 930  9570 930
 $Comp
-L Mechanical:MountingHole H1
+L Mechanical:MountingHole_Pad H1
 U 1 1 5DD609E4
-P 4000 4900
-F 0 "H1" H 4100 4946 50  0000 L CNN
-F 1 "MountingHole" H 4100 4855 50  0000 L CNN
-F 2 "" H 4000 4900 50  0001 C CNN
-F 3 "~" H 4000 4900 50  0001 C CNN
-	1    4000 4900
+P 4000 4820
+F 0 "H1" H 4100 4869 50  0000 L CNN
+F 1 "MountingHole" H 4100 4778 50  0000 L CNN
+F 2 "Mounting_Holes:MountingHole_2.2mm_M2_Pad" H 4000 4820 50  0001 C CNN
+F 3 "~" H 4000 4820 50  0001 C CNN
+	1    4000 4820
 	1    0    0    -1
 $EndComp
 $Comp
-L Mechanical:MountingHole H4
+L Mechanical:MountingHole_Pad H4
 U 1 1 5DD61216
-P 4740 5100
-F 0 "H4" H 4840 5146 50  0000 L CNN
-F 1 "MountingHole" H 4840 5055 50  0000 L CNN
-F 2 "" H 4740 5100 50  0001 C CNN
-F 3 "~" H 4740 5100 50  0001 C CNN
-	1    4740 5100
+P 4740 5270
+F 0 "H4" H 4840 5319 50  0000 L CNN
+F 1 "MountingHole" H 4840 5228 50  0000 L CNN
+F 2 "Mounting_Holes:MountingHole_2.2mm_M2_Pad" H 4740 5270 50  0001 C CNN
+F 3 "~" H 4740 5270 50  0001 C CNN
+	1    4740 5270
 	1    0    0    -1
 $EndComp
 $Comp
-L Mechanical:MountingHole H2
+L Mechanical:MountingHole_Pad H2
 U 1 1 5DD6158B
-P 4740 4910
-F 0 "H2" H 4840 4956 50  0000 L CNN
-F 1 "MountingHole" H 4840 4865 50  0000 L CNN
-F 2 "" H 4740 4910 50  0001 C CNN
-F 3 "~" H 4740 4910 50  0001 C CNN
-	1    4740 4910
+P 4740 4810
+F 0 "H2" H 4840 4859 50  0000 L CNN
+F 1 "MountingHole" H 4840 4768 50  0000 L CNN
+F 2 "Mounting_Holes:MountingHole_2.2mm_M2_Pad" H 4740 4810 50  0001 C CNN
+F 3 "~" H 4740 4810 50  0001 C CNN
+	1    4740 4810
 	1    0    0    -1
 $EndComp
 $Comp
-L Mechanical:MountingHole H3
+L Mechanical:MountingHole_Pad H3
 U 1 1 5DD62790
-P 4000 5110
-F 0 "H3" H 4100 5156 50  0000 L CNN
-F 1 "MountingHole" H 4100 5065 50  0000 L CNN
-F 2 "" H 4000 5110 50  0001 C CNN
-F 3 "~" H 4000 5110 50  0001 C CNN
-	1    4000 5110
+P 4000 5280
+F 0 "H3" H 4100 5329 50  0000 L CNN
+F 1 "MountingHole" H 4100 5238 50  0000 L CNN
+F 2 "Mounting_Holes:MountingHole_2.2mm_M2_Pad" H 4000 5280 50  0001 C CNN
+F 3 "~" H 4000 5280 50  0001 C CNN
+	1    4000 5280
 	1    0    0    -1
 $EndComp
@@
 Text Notes 4020 4590 0    173  ~ 0
 Mounting\nHoles
+$Comp
+L power:GND #PWR?
+U 1 1 5DDE94B5
+P 4000 4950
+F 0 "#PWR?" H 4000 4700 50  0001 C CNN
+F 1 "GND" H 4130 4900 50  0000 C CNN
+F 2 "" H 4000 4950 50  0001 C CNN
+F 3 "" H 4000 4950 50  0001 C CNN
+	1    4000 4950
+	1    0    0    -1
+$EndComp
+Wire Wire Line
+	4000 4950 4000 4920
+$Comp
+L power:GND #PWR?
+U 1 1 5DE03493
+P 4740 4940
+F 0 "#PWR?" H 4740 4690 50  0001 C CNN
+F 1 "GND" H 4870 4890 50  0000 C CNN
+F 2 "" H 4740 4940 50  0001 C CNN
+F 3 "" H 4740 4940 50  0001 C CNN
+	1    4740 4940
+	1    0    0    -1
+$EndComp
+Wire Wire Line
+	4740 4940 4740 4910
+$Comp
+L power:GND #PWR?
+U 1 1 5DE0C81A
+P 4740 5410
+F 0 "#PWR?" H 4740 5160 50  0001 C CNN
+F 1 "GND" H 4870 5360 50  0000 C CNN
+F 2 "" H 4740 5410 50  0001 C CNN
+F 3 "" H 4740 5410 50  0001 C CNN
+	1    4740 5410
+	1    0    0    -1
+$EndComp
+Wire Wire Line
+	4740 5410 4740 5370
+$Comp
+L power:GND #PWR?
+U 1 1 5DE15A51
+P 4000 5410
+F 0 "#PWR?" H 4000 5160 50  0001 C CNN
+F 1 "GND" H 4130 5360 50  0000 C CNN
+F 2 "" H 4000 5410 50  0001 C CNN
+F 3 "" H 4000 5410 50  0001 C CNN
+	1    4000 5410
+	1    0    0    -1
+$EndComp
+Wire Wire Line
+	4000 5410 4000 5380
 $EndSCHEMATC

Commit message: Committed V1.1
Parts:
- removed J2: GPIO Conn, Pin_Headers:Pin_Header_Straight_1x04_Pitch2.54mm, symbol Connector_Generic:Conn_01x04
- removed J3: Flash Programming Header, Pin_Headers:Pin_Header_Straight_2x06_Pitch2.00mm, symbol Connector_Generic:Conn_02x05_Counter_Clockwise
- added FID1, FID2, FID3: Fiducial, Fiducials:Fiducial_1mm_Dia_2.54mm_Outer_CopperTop, symbol Mechanical:Fiducial
- added J2: GPIO_header, Pin_Headers:Pin_Header_Straight_1x02_Pitch2.54mm, symbol Connector_Generic:Conn_01x02
- added J3: Programing Header, Pin_Headers:Pin_Header_Straight_2x04_Pitch2.00mm, symbol Connector_Generic:Conn_02x04_Odd_Even
- C5: value C -> 0.1uF
- D1: value LED -> LTST-C191KRKT
- D2, D5: value LED -> LTST-C191KGKT
- D3: value D_TVS -> VESD05A1-02V-G-08
- D4: value D_Zener -> BZT585B3V3T-7
- D6: value LED -> L130-5780001400001
- D7: value D_TVS -> ESD5Z3.3T1G
- JP1, JP2, JP3: value N/A -> RC0402JR-070RL
- U3: footprint TO_SOT_Packages_SMD:SOT-23 -> TO_SOT_Packages_SMD:Texas_DRT-3
Connections:
- net 3.3V: now also J3.1 (Pin_1)
- net AS_RST: now also D8.3 (IO2), J3.3 (Pin_3); no longer D8.1 (IO1)
- net CS: now also D8.4 (IO3), J3.2 (Pin_2); no longer D8.6 (IO5)
- net GND: now also J3.5 (Pin_5), J3.7 (Pin_7)
- net GP2: now also J2.1 (Pin_1)
- net GP3: now also J2.2 (Pin_2)
- net MISO: now also D8.1 (IO1), J3.8 (Pin_8); no longer D8.4 (IO3)
- net MOSI: now also D8.6 (IO5), J3.6 (Pin_6); no longer D8.3 (IO2)
- net SCK: now also J3.4 (Pin_4)
- net USB_-: now reaches J1.2 (D-), R2.2, U3.2 (D-)
- net USB_+: now reaches J1.3 (D+), R1.2, U3.1 (D+)
- net D_-: now reaches R2.1, U1.12 (D-)
- net D_+: now reaches R1.1, U1.13 (D+)
