File: low_cost_multispectral_sensor/_saved_low_cost_multispectral_sensor.sch (KiCad schematic (older format))
At the start: 41 parts, among them J1 USB_B_Micro, J2 GPIO Conn, J3 Flash Programming Header, U1 MCP2221, U2 MIC5219-3.3YMM, U3 TPD2EUSB30, U5 AS726x, U7 AT25SF041

Commit message: Initial layout completion
Parts:
- H1, H2, H3, H4: footprint (none) -> Mounting_Holes:MountingHole_2.2mm_M2_Pad
Changed lines of the file:
@@
 F 0 "H1" H 4100 4946 50  0000 L CNN
 F 1 "MountingHole" H 4100 4855 50  0000 L CNN
-F 2 "" H 4000 4900 50  0001 C CNN
+F 2 "Mounting_Holes:MountingHole_2.2mm_M2_Pad" H 4000 4900 50  0001 C CNN
 F 3 "~" H 4000 4900 50  0001 C CNN
 	1    4000 4900
@@
 F 0 "H4" H 4840 5146 50  0000 L CNN
 F 1 "MountingHole" H 4840 5055 50  0000 L CNN
-F 2 "" H 4740 5100 50  0001 C CNN
+F 2 "Mounting_Holes:MountingHole_2.2mm_M2_Pad" H 4740 5100 50  0001 C CNN
 F 3 "~" H 4740 5100 50  0001 C CNN
 	1    4740 5100
@@
 F 0 "H2" H 4840 4956 50  0000 L CNN
 F 1 "MountingHole" H 4840 4865 50  0000 L CNN
-F 2 "" H 4740 4910 50  0001 C CNN
+F 2 "Mounting_Holes:MountingHole_2.2mm_M2_Pad" H 4740 4910 50  0001 C CNN
 F 3 "~" H 4740 4910 50  0001 C CNN
 	1    4740 4910
@@
 F 0 "H3" H 4100 5156 50  0000 L CNN
 F 1 "MountingHole" H 4100 5065 50  0000 L CNN
-F 2 "" H 4000 5110 50  0001 C CNN
+F 2 "Mounting_Holes:MountingHole_2.2mm_M2_Pad" H 4000 5110 50  0001 C CNN
 F 3 "~" H 4000 5110 50  0001 C CNN
 	1    4000 5110
