File: low_cost_multispectral_sensor/low_cost_multispectral_sensor.kicad_pcb (KiCad board)
At the start: 4 copper layers, 39.8 x 39.8 mm, 41 parts, among them J1 USB_B_Micro, J2 GPIO Conn, J3 Flash Programming Header, U1 MCP2221, U2 MIC5219-3.3YMM, U3 TPD2EUSB30, U5 AS726x, U7 AT25SF041

Commit message: update
Connections:
- H1 pad 1: (no net) -> GND
- H2 pad 1: (no net) -> GND
- H3 pad 1: (no net) -> GND
- H4 pad 1: (no net) -> GND
Routing:
- net GND: track 35.0 -> 32.3 mm
Other:
- board text added: "Low Cost USB Multispectral Sensor Version 1.0"
Changed lines of the file:
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@@
   (general
     (thickness 1.6)
-    (drawings 18)
-    (tracks 387)
+    (drawings 19)
+    (tracks 385)
     (zones 0)
     (modules 41)
@@
   (layers
     (0 F.Cu signal)
-    (1 In1.Cu power)
-    (2 In2.Cu power)
-    (31 B.Cu signal)
+    (1 In1.Cu power hide)
+    (2 In2.Cu power hide)
+    (31 B.Cu signal hide)
     (32 B.Adhes user)
     (33 F.Adhes user)
@@
   )
   (module Mounting_Holes:MountingHole_2.2mm_M2_Pad (layer F.Cu)
-    (at 139.775 74.1 180)
-    (descr "Mounting Hole 2.2mm, M2")
-    (tags "mounting hole 2.2mm m2")
-    (attr virtual)
-    (fp_text reference H1 (at 0 -3.2 180) (layer F.SilkS)
-      (effects (font (size 1 1) (thickness 0.15)))
-    )
-    (fp_text value MountingHole (at 3.25 3.9 180) (layer F.Fab)
-      (effects (font (size 1 1) (thickness 0.15)))
-    )
-    (fp_circle (center 0 0) (end 2.45 0) (layer F.CrtYd) (width 0.05))
-    (fp_circle (center 0 0) (end 2.2 0) (layer Cmts.User) (width 0.15))
-    (fp_text user %R (at 0.3 0 180) (layer F.Fab)
-      (effects (font (size 1 1) (thickness 0.15)))
-    )
-    (pad 1 thru_hole circle (at 0 0 180) (size 4.4 4.4) (drill 2.2) (layers *.Cu *.Mask))
-  )
-  (module Mounting_Holes:MountingHole_2.2mm_M2_Pad (layer F.Cu)
     (at 139.775 108.25)
     (descr "Mounting Hole 2.2mm, M2")
@@
       (effects (font (size 1 1) (thickness 0.15)))
     )
-    (pad 1 thru_hole circle (at 0 0) (size 4.4 4.4) (drill 2.2) (layers *.Cu *.Mask))
+    (pad 1 thru_hole circle (at 0 0) (size 4.4 4.4) (drill 2.2) (layers *.Cu *.Mask)
+      (net 1 GND))
   )
   (module Mounting_Holes:MountingHole_2.2mm_M2_Pad (layer F.Cu)
@@
     (fp_circle (center 0 0) (end 2.2 0) (layer Cmts.User) (width 0.15))
     (fp_circle (center 0 0) (end 2.45 0) (layer F.CrtYd) (width 0.05))
-    (pad 1 thru_hole circle (at 0 0) (size 4.4 4.4) (drill 2.2) (layers *.Cu *.Mask))
+    (pad 1 thru_hole circle (at 0 0) (size 4.4 4.4) (drill 2.2) (layers *.Cu *.Mask)
+      (net 1 GND))
   )
   (module Mounting_Holes:MountingHole_2.2mm_M2_Pad (layer F.Cu)
@@
     (fp_circle (center 0 0) (end 2.2 0) (layer Cmts.User) (width 0.15))
     (fp_circle (center 0 0) (end 2.45 0) (layer F.CrtYd) (width 0.05))
-    (pad 1 thru_hole circle (at 0 0 180) (size 4.4 4.4) (drill 2.2) (layers *.Cu *.Mask))
+    (pad 1 thru_hole circle (at 0 0 180) (size 4.4 4.4) (drill 2.2) (layers *.Cu *.Mask)
+      (net 1 GND))
+  )
+  (module Mounting_Holes:MountingHole_2.2mm_M2_Pad (layer F.Cu)
+    (at 139.775 74.1 180)
+    (descr "Mounting Hole 2.2mm, M2")
+    (tags "mounting hole 2.2mm m2")
+    (attr virtual)
+    (fp_text reference H1 (at 0 -3.2 180) (layer F.SilkS)
+      (effects (font (size 1 1) (thickness 0.15)))
+    )
+    (fp_text value MountingHole (at 0 3.2 180) (layer F.Fab)
+      (effects (font (size 1 1) (thickness 0.15)))
+    )
+    (fp_circle (center 0 0) (end 2.45 0) (layer F.CrtYd) (width 0.05))
+    (fp_circle (center 0 0) (end 2.2 0) (layer Cmts.User) (width 0.15))
+    (fp_text user %R (at 0.3 0 180) (layer F.Fab)
+      (effects (font (size 1 1) (thickness 0.15)))
+    )
+    (pad 1 thru_hole circle (at 0 0 180) (size 4.4 4.4) (drill 2.2) (layers *.Cu *.Mask)
+      (net 1 GND))
+  )
+  (gr_text "Low Cost USB \nMultispectral Sensor \nVersion 1.0 " (at 146.625 83.925) (layer F.SilkS)
+    (effects (font (size 0.75 0.75) (thickness 0.15)))
   )
   (gr_text GND (at 167.075 101.7) (layer B.SilkS)
@@
     (effects (font (size 0.5 0.5) (thickness 0.1)) (justify mirror))
   )
-  (gr_text MISO (at 173.75 93.475) (layer B.SilkS)
+  (gr_text MISO (at 173.775 93.45) (layer B.SilkS)
     (effects (font (size 0.5 0.5) (thickness 0.1)) (justify mirror))
   )
@@
     (effects (font (size 0.5 0.5) (thickness 0.1)) (justify mirror))
   )
-  (gr_text GP3 (at 143.6 93.525) (layer B.SilkS)
-    (effects (font (size 1.5 1.5) (thickness 0.3)) (justify mirror))
-  )
-  (gr_text GP2 (at 143.55 91.075) (layer B.SilkS)
-    (effects (font (size 1.5 1.5) (thickness 0.3)) (justify mirror))
-  )
-  (gr_text GP1 (at 143.5 88.575) (layer B.SilkS)
-    (effects (font (size 1.5 1.5) (thickness 0.3)) (justify mirror))
-  )
-  (gr_text GP0 (at 143.525 85.8) (layer B.SilkS)
-    (effects (font (size 1.5 1.5) (thickness 0.3)) (justify mirror))
+  (gr_text GP3 (at 142.775 93.475) (layer B.SilkS)
+    (effects (font (size 1 1) (thickness 0.25)) (justify mirror))
+  )
+  (gr_text GP2 (at 142.8 91) (layer B.SilkS)
+    (effects (font (size 1 1) (thickness 0.25)) (justify mirror))
+  )
+  (gr_text GP1 (at 142.85 88.325) (layer B.SilkS)
+    (effects (font (size 1 1) (thickness 0.25)) (justify mirror))
+  )
+  (gr_text GP0 (at 142.65 85.85) (layer B.SilkS)
+    (effects (font (size 1 1) (thickness 0.25)) (justify mirror))
   )
   (gr_line (start 136.625 71.25) (end 176.425 71.25) (layer Edge.Cuts) (width 0.05))
@@
   (via (at 152.325 98.175) (size 0.8) (drill 0.4) (layers F.Cu B.Cu) (net 1))
   (segment (start 152.325 97.1) (end 152.325 98.175) (width 0.25) (layer F.Cu) (net 1))
-  (segment (start 153.625 108.4) (end 152.525 108.4) (width 0.5) (layer F.Cu) (net 1))
-  (segment (start 152.525 108.4) (end 150.925 108.4) (width 0.5) (layer F.Cu) (net 1))
   (segment (start 158.25 104.025) (end 158.525 104.025) (width 0.25) (layer F.Cu) (net 1))
   (segment (start 157.825 106.95) (end 157.825 104.45) (width 0.25) (layer F.Cu) (net 1))

Commit message: Committed V1.1
Parts:
- added FID1: Fiducial, Fiducials:Fiducial_1mm_Dia_2.54mm_Outer_CopperTop, F.Cu at (139.8, 80.5)
- added FID2: Fiducial, Fiducials:Fiducial_1mm_Dia_2.54mm_Outer_CopperTop, F.Cu at (139.6, 102.1)
- added FID3: Fiducial, Fiducials:Fiducial_1mm_Dia_2.54mm_Outer_CopperTop, F.Cu at (165.8, 108.7)
- C5: value C -> 0.1uF
- D1: value LED -> LTST-C191KRKT
- D2, D5: value LED -> LTST-C191KGKT
- D3: value D_TVS -> VESD05A1-02V-G-08
- D4: value D_Zener -> BZT585B3V3T-7
- D6: value LED -> L130-5780001400001
- D7: value D_TVS -> ESD5Z3.3T1G
- J2: value GPIO Conn -> GPIO_header; footprint Pin_Headers:Pin_Header_Straight_1x04_Pitch2.54mm -> Pin_Headers:Pin_Header_Straight_1x02_Pitch2.54mm
- J3: value Flash Programming Header -> Programing Header; footprint Pin_Headers:Pin_Header_Straight_2x06_Pitch2.00mm -> Pin_Headers:Pin_Header_Straight_2x04_Pitch2.00mm
- JP1, JP2, JP3: value N/A -> RC0402JR-070RL
- U3: footprint TO_SOT_Packages_SMD:SOT-23 -> TO_SOT_Packages_SMD:Texas_DRT-3
- moved D8 8.51 mm to (170.3, 94.0)
- moved J2 5.11 mm to (139.7, 91.1)
- moved J3 4.13 mm to (167.2, 101.1), turned to 90 degrees
- moved C10 1.27 mm to (165.6, 79.7)
- moved JP3 1.27 mm to (170.2, 87.3)
- moved R10 1.27 mm to (170.2, 86.2)
- moved R9 1.27 mm to (167.7, 76.4)
- moved U7 1.27 mm to (169.1, 81.0)
- moved U3 0.68 mm to (156.2, 101.4), turned to 180 degrees
- moved R1 0.62 mm to (157.2, 97.8)
Connections:
- net Net-(J1-Pad2) renamed /USB_-
- net Net-(J1-Pad3) renamed /USB_+
- net Net-(R1-Pad1) renamed /D_+
- net Net-(R2-Pad1) renamed /D_-
- D8 pad 1: /AS_RST -> /MISO
- D8 pad 3: /MOSI -> /AS_RST
- D8 pad 4: /MISO -> /CS
- D8 pad 6: /CS -> /MOSI
- J2 pad 1: /GP0 -> /GP2
- J2 pad 2: /GP1 -> /GP3
- J3 pad 1: GND -> /3.3V
- J3 pad 2: GND -> /CS
- J3 pad 3: GND -> /AS_RST
- J3 pad 4: /AS_RST -> /SCK
- J3 pad 6: /CS -> /MOSI
- J3 pad 7: /SCK -> GND
- J3 pad 8: /MOSI -> /MISO
Routing:
- net /GP0: track 29.4 -> 2.08 mm, vias 1 -> 0
- net /MISO: track 56.8 -> 33.0 mm, vias 0 -> 2
- net /GP1: track 25.4 -> 4.32 mm, vias 1 -> 0
- net /SCK: track 67.4 -> 46.4 mm, vias 3 -> 1
- net /AS_RST: track 33.1 -> 48.8 mm, vias 2 -> 3
- net /CS: track 36.6 -> 28.0 mm, vias 3 -> 2
- net /TX: track 28.8 -> 20.5 mm
- net /RX: track 23.9 -> 17.4 mm
- net /3.3V: track 38.5 -> 40.5 mm, vias 11 -> 12
- net GND: track 32.3 -> 30.7 mm
- net Net-(D5-Pad1): track 8.36 -> 9.88 mm
- net /USB_-: track 10.1 -> 9.38 mm
- net /MOSI: track 50.4 -> 49.7 mm, vias 4 -> 1
- net /VUSB: track 4.39 -> 4.95 mm
Other:
- board text added: "Low Cost USB Multispectral Sensor Version 1.1"
- board text removed: "GP0"
- board text removed: "GP1"
- board text removed: "Low Cost USB Multispectral Sensor Version 1.0"
